File: AleeMacro.kicad_pcb (KiCad board)
At the start: 2 copper layers, 245.1 x 103.6 mm, 67 parts, among them SW1 SW_Push, U1 ProMicro

Commit message: LED Traces Confirmed
Parts:
- removed the ? at (181.9, 87.9)
- moved D10 1.75 mm to (173.2, 79.2)
Routing:
- net (no net): track 0.00 -> 98.4 mm
- net GND: track 45.0 -> 33.8 mm
- net ROW3: track 104.2 -> 106.0 mm
- net ROW2: track 64.3 -> 65.7 mm
- net SCL: track 26.5 -> 27.8 mm
- net Net-(D12-Pad2): track 10.9 -> 9.66 mm

Commit message: Prototype Run 1
Parts:
- LEDstrip (NoJump): renamed from LED Strip (No Jump)
Routing:
- net (no net): track 98.4 -> 117.8 mm
- net ROW1: track 78.4 -> 79.1 mm
